Commit message: Modify left/right joint axis

File: xacro/modelc.xacro (robot description, xacro)
@@ -1,4 +1,4 @@
 <?xml version="1.0"?>
-<robot xmlns:xacro="http://www.ros.org/wiki/xacro" name="whill_modelc" >
+<robot xmlns:xacro="http://www.ros.org/wiki/xacro" name="whill" >
     <link name="base_link">
     </link>
@@ -30,5 +30,5 @@
         <origin xyz="0.3 0 0.0" rpy="0 0 0"/>
     </joint>
-    <link name="footrest_link">
+    <link name="footrest_link">imu_joint
         <collision>
             <geometry>
@@ -80,5 +80,5 @@
         <child link="left_wheel_link" />
         <origin xyz="-0.3 0.245 0" rpy="-1.57 0 0" />
-        <axis xyz="0 0 1" />
+        <axis xyz="0 0 -1" />
     </joint>
     <link name="right_wheel_link">
@@ -177,4 +177,5 @@
         <actuator name="right_wheel_motor">
             <hardwareInterface>hardware_interface/VelocityJointInterface</hardwareInterface>
+            <!-- <mechanicalReduction>30</mechanicalReduction> -->
             <mechanicalReduction>30</mechanicalReduction>
         </actuator>
@@ -187,4 +188,5 @@
         <actuator name="left_wheel_motor">
             <hardwareInterface>hardware_interface/VelocityJointInterface</hardwareInterface>
+            <!-- <mechanicalReduction>30</mechanicalReduction> -->
             <mechanicalReduction>30</mechanicalReduction>
         </actuator>
@@ -194,4 +196,5 @@
         <plugin name="gazebo_ros_control" filename="libgazebo_ros_control.so">
             <robotNamespace>/whill_simulator</robotNamespace>
+            <legacyModeNS>true</legacyModeNS>
         </plugin>
     </gazebo>
@@ -201,21 +204,19 @@
         <mu2 value="0.05" />
     </gazebo>
-    <gazebo reference="sensor_arm_link">
-        <selfCollide>true</selfCollide>
-        <mu1 value="0.05" />
-        <mu2 value="0.05" />
-    </gazebo>
-    <gazebo reference="rearwheel_right">
-        <selfCollide>true</selfCollide>
-        <mu1 value="1.0" />
-        <mu2 value="1.0" />
-    </gazebo>
-    <gazebo reference="rearwheel_left">
-        <selfCollide>true</selfCollide>
-        <mu1 value="1.0" />
-        <mu2 value="1.0" />
+    <gazebo reference="right_wheel_link">
+        <selfCollide>true</selfCollide>
+        <material>Gazebo/Gray</material>
+        <mu1 value="0.8" />
+        <mu2 value="0.8" />
+    </gazebo>
+    <gazebo reference="left_wheel_link">
+        <selfCollide>true</selfCollide>
+        <material>Gazebo/Gray</material>
+        <mu1 value="0.8" />
+        <mu2 value="0.8" />
     </gazebo>
     <gazebo reference="frontwheel_right">
         <selfCollide>true</selfCollide>
+        <material>Gazebo/Gray</material>
         <mu1 value="0.0" />
         <mu2 value="0.0" />
@@ -223,4 +224,5 @@
     <gazebo reference="frontwheel_left">
         <selfCollide>true</selfCollide>
+        <material>Gazebo/Gray</material>
         <mu1 value="0.0" />
         <mu2 value="0.0" />

Commit message: Modify xacro file

File: xacro/modelc.xacro (robot description, xacro)
@@ -132,5 +132,5 @@
         <child link="frontwheel_left" />
         <origin xyz="0.3 -0.245 0" rpy="1.57 0 0" />
-        <axis xyz="0 0 1" />
+        <axis xyz="0 0 -1" />
     </joint>
     <link name="frontwheel_right">
@@ -158,5 +158,5 @@
         <child link="frontwheel_right"/>
         <origin xyz="0.3 0.245 0" rpy="1.57 0 0" />
-        <axis xyz="0 0 -1" />
+        <axis xyz="0 0 1" />
     </joint>
     <!-- IMU -->
@@ -169,4 +169,10 @@
         <child link="imu"/>
     </joint>
+    <!-- <joint name="imu_joint" type="fixed">
+        <axis xyz="0 1 0" />
+        <origin xyz="0.02 0 0.05" rpy="0 0.85521133347 3.14159265359"/>
+        <parent link="base_floor"/>
+        <child link="imu"/>
+    </joint> -->
     <!-- ===============  Transmission =============== -->
     <transmission name="right_wheel_trans">

Commit message: Change rolling angle of right/left wheel

File: xacro/modelc.xacro (robot description, xacro)
@@ -79,5 +79,5 @@
         <parent link="base_floor" />
         <child link="left_wheel_link" />
-        <origin xyz="-0.3 0.245 0" rpy="-1.57 0 0" />
+        <origin xyz="-0.3 0.245 0" rpy="1.57 0 0" />
         <axis xyz="0 0 -1" />
     </joint>
@@ -105,5 +105,5 @@
         <parent link="base_floor" />
         <child link="right_wheel_link" />
-        <origin xyz="-0.3 -0.245 0" rpy="1.57 0 0" />
+        <origin xyz="-0.3 -0.245 0" rpy="-1.57 0 0" />
         <axis xyz="0 0 1" />
     </joint>

Commit message: Add camera to the model

File: xacro/modelc.xacro (robot description, xacro)
@@ -30,5 +30,5 @@
         <origin xyz="0.3 0 0.0" rpy="0 0 0"/>
     </joint>
-    <link name="footrest_link">imu_joint
+    <link name="footrest_link">
         <collision>
             <geometry>
@@ -160,19 +160,74 @@
         <axis xyz="0 0 1" />
     </joint>
-    <!-- IMU -->
+     <!-- ===============  IMU =============== -->
     <link name="imu">
+    <visual>
+        <origin xyz="0 0 0" rpy="0 0 0" />
+            <geometry>
+                <box size="0.02 0.02 0.02"/>
+            </geometry>
+            <material name="Blue" />
+        </visual>
     </link>
     <joint name="imu_joint" type="fixed">
+        <parent link="base_floor"/>
+        <child link="imu"/>
         <axis xyz="0 1 0" />
         <origin xyz="0.02 0 0.05" rpy="0 0.85521133347 3.14159265359"/>
-        <parent link="base_link"/>
-        <child link="imu"/>
-    </joint>
-    <!-- <joint name="imu_joint" type="fixed">
-        <axis xyz="0 1 0" />
-        <origin xyz="0.02 0 0.05" rpy="0 0.85521133347 3.14159265359"/>
-        <parent link="base_floor"/>
-        <child link="imu"/>
-    </joint> -->
+    </joint>
+    <!-- =============== Sensor =============== -->
+    <!-- =============== Camera =============== -->
+    <link name="camera_link">
+    <visual>
+      <origin xyz="0 0 0" rpy="0 0 0" />
+      <geometry>
+        <box size="0.05 0.1 0.05"/>
+      </geometry>
+      <material name="Blue" />
+    </visual>
+  </link>
+  <joint name="camera_joint" type="fixed">
+    <parent link="base_floor"/>
+    <child link="camera_link" />
+    <origin xyz="0.3 0 0.2" rpy="0 0 0" />
+  </joint>
+  <gazebo reference="camera_link">
+    <material>Gazebo/Blue</material>
+    <turnGravityOff>false</turnGravityOff>
+    <sensor type="camera" name="camera1">
+      <update_rate>15.0</update_rate>
+      <camera name="head">
+          <pose>0 0 0 0 0 0</pose>
+        <horizontal_fov>1.3962634</horizontal_fov>
+        <image>
+          <width>400</width>
+          <height>400</height>
+          <format>R8G8B8</format>
+        </image>
+        <clip>
+          <near>0.01</near>
+          <far>100</far>
+        </clip>
+        <noise>
+          <type>gaussian</type>
+          <stddev>0.007</stddev>
+        </noise>
+      </camera>
+      <plugin name="camera_controller" filename="libgazebo_ros_camera.so">
+        <alwaysOn>true</alwaysOn>
+        <updateRate>0.0</updateRate>
+        <cameraName>whill_simulator/camera1</cameraName>
+        <imageTopicName>image_raw</imageTopicName>
+        <cameraInfoTopicName>camera_info</cameraInfoTopicName>
+        <frameName>camera_link</frameName>
+        <hackBaseline>0.07</hackBaseline>
+        <distortionK1>0.0</distortionK1>
+        <distortionK2>0.0</distortionK2>
+        <distortionK3>0.0</distortionK3>
+        <distortionT1>0.0</distortionT1>
+        <distortionT2>0.0</distortionT2>
+      </plugin>
+    </sensor>
+  </gazebo>
     <!-- ===============  Transmission =============== -->
     <transmission name="right_wheel_trans">
@@ -198,5 +253,5 @@
         </actuator>
     </transmission>
-    <!-- For Gazebo -->
+    <!-- ===============  Gazebo =============== -->
     <gazebo>
         <plugin name="gazebo_ros_control" filename="libgazebo_ros_control.so">

Commit message: Add Rplidar to xacro file

File: xacro/modelc.xacro (robot description, xacro)
@@ -230,4 +230,51 @@
     </sensor>
   </gazebo>
+    <!-- =============== LiDAR =============== -->
+    <link name="lidar_link">
+        <visual>
+        <origin xyz="0 0 0" rpy="0 0 0" />
+        <geometry>
+            <box size="0.1 0.1 0.1"/>
+        </geometry>
+        <material name="Green" />
+        </visual>
+    </link>
+    <joint name="lidar_joint" type="fixed">
+        <parent link="base_floor"/>
+        <child link="lidar_link" />
+        <origin xyz="0.3 0 0.5" rpy="0 0 0" />
+    </joint>
+    <gazebo reference="lidar_link">
+        <material>Gazebo/Green</material>
+        <sensor type="ray" name="head_rplidar_sensor">
+            <pose>0 0 0 0 0 0</pose>
+            <visualize>false</visualize>
+            <update_rate>40</update_rate>
+            <ray>
+                <scan>
+                    <horizontal>
+                        <samples>720</samples>
+                        <resolution>1</resolution>
+                        <min_angle>-3.14159265</min_angle>
+                        <max_angle>3.14159265</max_angle>
+                    </horizontal>
+                </scan>
+                <range>
+                    <min>0.2</min>
+                    <max>12.0</max>
+                    <resolution>0.01</resolution>
+                </range>
+                <noise>
+                    <type>gaussian</type>
+                    <mean>0.0</mean>
+                    <stddev>0.01</stddev>
+                </noise>
+            </ray>
+            <plugin name="gazebo_ros_head_rplidar_controller" filename="libgazebo_ros_laser.so">
+                <topicName>scan</topicName>
+                <frameName>lidar_link</frameName>
+            </plugin>
+            </sensor>
+    </gazebo>
     <!-- ===============  Transmission =============== -->
     <transmission name="right_wheel_trans">
